Commit message: factory update: last dev

File: pybullet_tree_sim/urdf/end_effectors/mock_pruner/macro/mock_pruner_macro.urdf.xacro (robot description, xacro)
@@ -10,11 +10,11 @@
         <!-- static properties -->
         <xacro:property name="mock_pruner_mass" value="0.256" />
-        <xacro:property name="base__tool0_offset" value="0.0 0.0050825 0.1601525"/>
+        <xacro:property name="base__tool0_offset" value="0.0 0.0 0.2"/>
         <!-- <xacro:property name="base__tool0_offset" value="0.0 0.0 0.20"/> -->
-        <xacro:property name="base__tof0_offset" value="${tof0_offset}"/>
+        <xacro:property name="base__tof0_offset" value="-0.0 -0.0 0.1"/>
         <xacro:property name="base__tof1_offset" value="${tof1_offset}"/>
         <!-- <xacro:property name="base__tof0_offset" value="${tof0_offset} 0 0.15"/> -->
         <!-- <xacro:property name="base__tof1_offset" value="${tof1_offset} 0 0.15"/> -->
-        <xacro:property name="base__camera0_offset" value="-0.0017977 -0.0715747 0.0711646"/>
+        <xacro:property name="base__camera0_offset" value="-0.0 -0.0 0.1"/>
         <!-- additional args -->
         <xacro:arg name="rotation_correction_plate_prefix" default="rotation_correction_plate__" />
@@ -46,20 +46,20 @@
             <visual>
                 <material name="orange">
-                    <color rgba="${255/255} ${108/255} ${10/255} 1.0"/>
+                    <color rgba="${255/255} ${255/255} ${100/255} 1.0"/>
                 </material>
-                <origin xyz="0 0 0" rpy="0 0 0"/>
+                <origin xyz="-0.04 0.0 0.0" rpy="0 0 0"/>
                 <geometry>
-                    <mesh filename="${mesh_base_path}/end_effectors/mock_pruner/MockPruner.STL" />
+                    <mesh filename="${mesh_base_path}/end_effectors/mock_pruner/mk3_gripper.STL" scale="0.001 0.001 0.001" />
                 </geometry>
             </visual>
             <collision>
-                <origin xyz="0 0 0" rpy="0 0 0"/>
+                <origin xyz="-0.04 0.0 0.0" rpy="0 0 0"/>
                 <geometry>
-                    <mesh filename="${mesh_base_path}/end_effectors/mock_pruner/MockPruner.STL" />
+                    <mesh filename="${mesh_base_path}/end_effectors/mock_pruner/mk3_gripper.STL" scale="0.001 0.001 0.001" />
                 </geometry>
             </collision>
             <inertial>
                 <mass value="${mock_pruner_mass}"/>
-                <origin xyz="0.0 0.0 0.0"/>
+                <origin xyz="0.0 0.0 0.05"/>
                 <inertia ixx="0.1" ixy="0.0" ixz="0.0" iyy="0.1" iyz="0.0" izz="0.1"/>
             </inertial>

File: pybullet_tree_sim/urdf/tmp/robot.urdf (robot description, URDF)
Before this commit: robot pruning_robot, 30 links, 29 joints
Links:
- link amiga__body: geometry collision box size=0.25 0.25 0.25; collision box size=1.132 0.6 0.2
- link dovetail_female_mount__body: geometry collision mesh filename=/home/rob/Codes/UR5-ApplePathPlanning-Sim-PyBullet/pybullet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; visual mesh filename=/home/rob/Codes/UR5-ApplePathPlanning-Sim-PyBullet/pybullet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
- link dovetail_male_mount__body: geometry collision mesh filename=/home/rob/Codes/UR5-ApplePathPlanning-Sim-PyBullet/pybullet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; visual mesh filename=/home/rob/Codes/UR5-ApplePathPlanning-Sim-PyBullet/pybullet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
- link mock_pruner__base: geometry collision mesh filename=/home/rob/Codes/UR5-ApplePathPlanning-Sim-PyBullet/pybullet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 scale=0.001 0.001 0.001; visual mesh filename=/home/rob/Codes/UR5-ApplePathPlanning-Sim-PyBullet/pybullet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 scale=0.001 0.001 0.001
- link rotation_correction_plate__body: geometry collision mesh filename=/home/rob/Codes/UR5-ApplePathPlanning-Sim-PyBullet/pybullet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; visual mesh filename=/home/rob/Codes/UR5-ApplePathPlanning-Sim-PyBullet/pybullet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
Joints:
- joint mock_pruner__base--camera0: origin xyz=-0.0017977 -0.0715747 0.0711646 rpy=0 0 0 -> xyz=-0.0 -0.0 0.1 rpy=0 0 0
- joint mock_pruner__base--tof0: origin xyz=0.10 -0.025 0.2 rpy=0 0 0 -> xyz=-0.0 -0.0 0.1 rpy=0 0 0
- joint mock_pruner__base--tool0: origin xyz=0.0 0.0050825 0.1601525 rpy=0 0 0 -> xyz=0.0 0.0 0.2 rpy=0 0 0

File: pybullet_tree_sim/urdf/trees/envy/macro/tree_base.urdf.xacro (robot description, xacro)
@@ -1,11 +1,12 @@
 <?xml version="1.0"?>
 <robot name="tree" xmlns:xacro="http://ros.org/wiki/xacro">
-    <xacro:macro name="tree" params="namespace tree_id tree_type parent *origin">
-        <xacro:include filename="./macro/tree_macro.urdf.xacro"/> <!-- TODO: get absolute file paths? -->
+    <xacro:macro name="tree" params="namespace tree_id tree_type parent use_visual_material:=true *origin">
+        <xacro:include filename="./macro/tree_macro.urdf.xacro"/>
         <xacro:tree_macro
             namespace="${namespace}"
             tree_id="${tree_id}"
             tree_type="${tree_type}"
-            parent="${parent}" >
+            parent="${parent}"
+            use_visual_material="${use_visual_material}" >
             <xacro:insert_block name="origin"/>
         </xacro:tree_macro>

File: pybullet_tree_sim/urdf/trees/envy/macro/tree_macro.urdf.xacro (robot description, xacro)
@@ -6,4 +6,5 @@
         namespace
         parent:=^|world
+        use_visual_material:=true
         *origin
         ">
@@ -13,13 +14,16 @@
             <visual>
                 <geometry>
-                    <mesh filename="./meshes/trees/envy/unlabeled/obj/${namespace}_${tree_type}_${str(tree_id).zfill(5)}.obj" scale="${scale}"/>
+                    <mesh filename="../../../../meshes/trees/${tree_type}/unlabeled/obj/${namespace}_${tree_type}_${str(tree_id).zfill(5)}.obj" scale="${scale}"/>
                 </geometry>
-                <material name="LightGrey">
-                    <color rgba="0.7 0.7 0.7 1.0"/>
-                </material>
+                <!-- Omit material when false so PyBullet applies per-group map_Kd from OBJ/MTL (v2 export). -->
+                <xacro:if value="${ str(use_visual_material).lower() in ('true', '1', 'yes') }">
+                    <material name="LightGrey">
+                        <color rgba="0.7 0.7 0.7 1.0"/>
+                    </material>
+                </xacro:if>
             </visual>
             <collision concave="true">
                 <geometry>
-                    <mesh filename="./meshes/trees/envy/unlabeled/obj/${namespace}_${tree_type}_${str(tree_id).zfill(5)}.obj" scale="${scale}"/>
+                    <mesh filename="../../../../meshes/trees/${tree_type}/unlabeled/obj/${namespace}_${tree_type}_${str(tree_id).zfill(5)}.obj" scale="${scale}"/>
                 </geometry>
             </collision>

File: pybullet_tree_sim/urdf/trees/envy/tree.urdf.xacro (robot description, xacro)
@@ -6,4 +6,5 @@
     <xacro:arg name="tree_type" default="envy" />
     <xacro:arg name="parent" default="world" />
+    <xacro:arg name="use_visual_material" default="true" />
     <!-- <xacro:arg name="xyz" default="0.0 0.0 0.0"/>
     <xacro:arg name="rpy" default="0.0 0.0 0.0"/> -->
@@ -12,5 +13,6 @@
         tree_id="$(arg tree_id)"
         tree_type="$(arg tree_type)"
-        parent="$(arg parent)" >
+        parent="$(arg parent)"
+        use_visual_material="$(arg use_visual_material)" >
         <origin rpy="0.0 0.0 0.0" xyz="0.0 0.0 0.0"/>
     </xacro:tree>
