Commit message: Sim: portable robot.urdf with bundled meshes (no ROS or machine-specific paths)
robot.urdf referenced 19 meshes by absolute path: 14 from ROS 2 ur_description (/opt/ros/humble),
1 from a local ROS workspace (branch_detection_ws) and 4 from /home/rob/... . They are now copied to
urdf/tmp/robot_meshes/{ur5e,amiga,end_effectors} (26 MB, BSD-3 licenses included) and referenced by
relative path, which PyBullet resolves from the URDF's folder.
- Verified: identical geometry (meshes, scales, collision shapes, AABBs of all 30 links), loads
  from a copied folder, expert replay reproduces as before.
- tools/bundle_robot_meshes.py redoes this after regenerating robot.urdf from xacro (needs ROS 2);
  it is idempotent and reproduces this commit's URDF from the old one.

File: pybullet_tree_sim/urdf/tmp/robot.urdf (robot description, URDF)
Before this commit: robot pruning_robot, 30 links, 29 joints
Links:
- link amiga__body: geometry collision box size=0.25 0.25 0.25; collision box size=1.132 0.6 0.2
- link dovetail_female_mount__body: geometry collision mesh filename=robot_meshes/end_effectors/dovetail/DovetailFemale.STL; visual mesh filename=robot_meshes/end_effectors/dovetail/DovetailFemale.STL
- link dovetail_male_mount__body: geometry collision mesh filename=robot_meshes/end_effectors/dovetail/DovetailMale.STL; visual mesh filename=robot_meshes/end_effectors/dovetail/DovetailMale.STL
- link mock_pruner__base: geometry collision mesh filename=robot_meshes/end_effectors/mock_pruner/mk3_gripper.STL scale=0.001 0.001 0.001; visual mesh filename=robot_meshes/end_effectors/mock_pruner/mk3_gripper.STL scale=0.001 0.001 0.001
- link rotation_correction_plate__body: geometry collision mesh filename=robot_meshes/end_effectors/rotation_correction_plate/Rotati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; visual mesh filename=robot_meshes/end_effectors/rotation_correction_plate/Rotati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
- link ur5e__base_link_inertia: geometry collision mesh filename=robot_meshes/ur5e/collision/base.stl; visual mesh filename=robot_meshes/ur5e/visual/base.dae
- link ur5e__forearm_link: geometry collision mesh filename=robot_meshes/ur5e/collision/forearm.stl; visual mesh filename=robot_meshes/ur5e/visual/forearm.dae
- link ur5e__shoulder_link: geometry collision mesh filename=robot_meshes/ur5e/collision/shoulder.stl; visual mesh filename=robot_meshes/ur5e/visual/shoulder.dae
- link ur5e__upper_arm_link: geometry collision mesh filename=robot_meshes/ur5e/collision/upperarm.stl; visual mesh filename=robot_meshes/ur5e/visual/upperarm.dae
- link ur5e__wrist_1_link: geometry collision mesh filename=robot_meshes/ur5e/collision/wrist1.stl; visual mesh filename=robot_meshes/ur5e/visual/wrist1.dae
- link ur5e__wrist_2_link: geometry collision mesh filename=robot_meshes/ur5e/collision/wrist2.stl; visual mesh filename=robot_meshes/ur5e/visual/wrist2.dae
- link ur5e__wrist_3_link: geometry collision mesh filename=robot_meshes/ur5e/collision/wrist3.stl; visual mesh filename=robot_meshes/ur5e/visual/wrist3.dae
